Commit message: Add new STL files for wrist roll components in the SO101 arm description
- Added wrist_roll_follower_so101_v1.stl (1406 KB)
- Added wrist_roll_pitch_so101_v2.stl (2637 KB)

File: M4-Control/so_arm_ws/src/so_arm100_description/urdf/so_arm100.gazebo.xacro (robot description, xacro)
@@ -2,13 +2,11 @@
 <robot xmlns:xacro="http://www.ros.org/wiki/xacro">
   <!-- Gazebo material overrides -->
-  <gazebo reference="base_link"><material>Gazebo/DarkGrey</material></gazebo>
-  <gazebo reference="link1"><material>Gazebo/Grey</material></gazebo>
-  <gazebo reference="link2"><material>Gazebo/White</material></gazebo>
-  <gazebo reference="link3"><material>Gazebo/Grey</material></gazebo>
-  <gazebo reference="link4"><material>Gazebo/White</material></gazebo>
-  <gazebo reference="link5"><material>Gazebo/DarkGrey</material></gazebo>
-  <gazebo reference="gripper_base"><material>Gazebo/DarkGrey</material></gazebo>
-  <gazebo reference="gripper_left"><material>Gazebo/Orange</material></gazebo>
-  <gazebo reference="gripper_right"><material>Gazebo/Orange</material></gazebo>
+  <gazebo reference="base_link">      <material>Gazebo/Yellow</material></gazebo>
+  <gazebo reference="shoulder_link">  <material>Gazebo/DarkGrey</material></gazebo>
+  <gazebo reference="upper_arm_link"> <material>Gazebo/Yellow</material></gazebo>
+  <gazebo reference="lower_arm_link"> <material>Gazebo/Yellow</material></gazebo>
+  <gazebo reference="wrist_link">     <material>Gazebo/DarkGrey</material></gazebo>
+  <gazebo reference="gripper_link">   <material>Gazebo/DarkGrey</material></gazebo>
+  <gazebo reference="moving_jaw_link"><material>Gazebo/Yellow</material></gazebo>
   <!-- ZED2 camera plugin (simulated stereo + depth) -->
   <gazebo reference="zed2_left_camera_frame">

File: M4-Control/so_arm_ws/src/so_arm100_description/urdf/so_arm100.ros2_control.xacro (robot description, xacro)
@@ -5,9 +5,8 @@
       <plugin>gazebo_ros2_control/GazeboSystem</plugin>
     </hardware>
-    <!-- Arm joints -->
-    <joint name="joint1">
+    <joint name="shoulder_pan">
       <command_interface name="position">
-        <param name="min">-3.14159</param>
-        <param name="max"> 3.14159</param>
+        <param name="min">-1.91986</param>
+        <param name="max"> 1.91986</param>
       </command_interface>
       <state_interface name="position"/>
@@ -15,8 +14,8 @@
       <state_interface name="effort"/>
     </joint>
-    <joint name="joint2">
+    <joint name="shoulder_lift">
       <command_interface name="position">
-        <param name="min">-1.5708</param>
-        <param name="max"> 1.5708</param>
+        <param name="min">-1.74533</param>
+        <param name="max"> 1.74533</param>
       </command_interface>
       <state_interface name="position"/>
@@ -24,8 +23,8 @@
       <state_interface name="effort"/>
     </joint>
-    <joint name="joint3">
+    <joint name="elbow_flex">
       <command_interface name="position">
-        <param name="min">-2.094</param>
-        <param name="max"> 2.094</param>
+        <param name="min">-1.69</param>
+        <param name="max"> 1.69</param>
       </command_interface>
       <state_interface name="position"/>
@@ -33,8 +32,8 @@
       <state_interface name="effort"/>
     </joint>
-    <joint name="joint4">
+    <joint name="wrist_flex">
       <command_interface name="position">
-        <param name="min">-1.5708</param>
-        <param name="max"> 1.5708</param>
+        <param name="min">-1.65806</param>
+        <param name="max"> 1.65806</param>
       </command_interface>
       <state_interface name="position"/>
@@ -42,8 +41,8 @@
       <state_interface name="effort"/>
     </joint>
-    <joint name="joint5">
+    <joint name="wrist_roll">
       <command_interface name="position">
-        <param name="min">-3.14159</param>
-        <param name="max"> 3.14159</param>
+        <param name="min">-2.74385</param>
+        <param name="max"> 2.84121</param>
       </command_interface>
       <state_interface name="position"/>
@@ -51,18 +50,8 @@
       <state_interface name="effort"/>
     </joint>
-    <!-- Gripper -->
-    <joint name="gripper_left_joint">
+    <joint name="gripper">
       <command_interface name="position">
-        <param name="min">-0.025</param>
-        <param name="max"> 0.0</param>
-      </command_interface>
-      <state_interface name="position"/>
-      <state_interface name="velocity"/>
-      <state_interface name="effort"/>
-    </joint>
-    <joint name="gripper_right_joint">
-      <command_interface name="position">
-        <param name="min">-0.025</param>
-        <param name="max"> 0.0</param>
+        <param name="min">-0.174533</param>
+        <param name="max"> 1.74533</param>
       </command_interface>
       <state_interface name="position"/>

File: M4-Control/so_arm_ws/src/so_arm100_description/urdf/so_arm100.urdf.xacro (robot description, xacro)
@@ -1,39 +1,19 @@
 <?xml version="1.0"?>
 <robot xmlns:xacro="http://www.ros.org/wiki/xacro" name="so_arm100">
-  <!-- ========================================================
-       SO-ARM100  —  6-DOF + gripper
-       Joints: base_rotation, shoulder, elbow, wrist_pitch,
-               wrist_roll, jaw (2 mirrored fingers)
-       All dimensions in metres, masses in kg.
-  ======================================================== -->
-  <!-- Gazebo / ros2_control plugin -->
+  <!-- Gazebo / ros2_control plugins -->
   <xacro:include filename="$(find so_arm100_description)/urdf/so_arm100.gazebo.xacro"/>
   <xacro:include filename="$(find so_arm100_description)/urdf/so_arm100.ros2_control.xacro"/>
-  <!-- ───────── Materials ───────── -->
-  <material name="dark_grey">
-    <color rgba="0.2 0.2 0.2 1.0"/>
+  <xacro:property name="mesh_pkg" value="package://so_arm100_description/meshes"/>
+  <!-- ── Materials ─────────────────────────────────────────── -->
+  <material name="3d_printed">
+    <color rgba="1.0 0.82 0.12 1.0"/>
   </material>
-  <material name="light_grey">
-    <color rgba="0.7 0.7 0.7 1.0"/>
-  </material>
-  <material name="white">
-    <color rgba="0.9 0.9 0.9 1.0"/>
+  <material name="sts3215">
+    <color rgba="0.1 0.1 0.1 1.0"/>
   </material>
   <material name="black">
     <color rgba="0.05 0.05 0.05 1.0"/>
   </material>
-  <material name="orange">
-    <color rgba="1.0 0.5 0.0 1.0"/>
-  </material>
-  <!-- ───────── Macro: box inertia ───────── -->
-  <xacro:macro name="box_inertia" params="m x y z">
-    <inertial>
-      <mass value="${m}"/>
-      <inertia ixx="${m*(y*y+z*z)/12}" ixy="0" ixz="0"
-               iyy="${m*(x*x+z*z)/12}" iyz="0"
-               izz="${m*(x*x+y*y)/12}"/>
-    </inertial>
-  </xacro:macro>
-  <!-- ───────── World / base_footprint ───────── -->
+  <!-- ── World anchor ──────────────────────────────────────── -->
   <link name="world"/>
   <joint name="world_to_base" type="fixed">
@@ -42,191 +22,282 @@
     <origin xyz="0 0 0" rpy="0 0 0"/>
   </joint>
-  <!-- ───────── Base link ───────── -->
+  <!-- ── base_link ─────────────────────────────────────────── -->
   <link name="base_link">
-    <visual>
-      <origin xyz="0 0 0.025" rpy="0 0 0"/>
-      <geometry><cylinder radius="0.055" length="0.05"/></geometry>
-      <material name="dark_grey"/>
-    </visual>
-    <collision>
-      <origin xyz="0 0 0.025" rpy="0 0 0"/>
-      <geometry><cylinder radius="0.055" length="0.05"/></geometry>
-    </collision>
-    <xacro:box_inertia m="0.5" x="0.11" y="0.11" z="0.05"/>
-  </link>
-  <!-- ───────── Joint 1: Base rotation (yaw) ───────── -->
-  <joint name="joint1" type="revolute">
+    <inertial>
+      <origin xyz="0.0137179 -5.19711e-05 0.0334843" rpy="0 0 0"/>
+      <mass value="0.147"/>
+      <inertia ixx="0.000114686" ixy="-4.59787e-07" ixz="4.97151e-06"
+               iyy="0.000136117" iyz="9.75275e-08" izz="0.000130364"/>
+    </inertial>
+    <visual>
+      <origin xyz="-0.00636471 -9.94414e-05 -0.0024" rpy="1.5708 0 1.5708"/>
+      <geometry><mesh filename="${mesh_pkg}/base_motor_holder_so101_v1.stl"/></geometry>
+      <material name="3d_printed"/>
+    </visual>
+    <collision>
+      <origin xyz="-0.00636471 -9.94414e-05 -0.0024" rpy="1.5708 0 1.5708"/>
+      <geometry><mesh filename="${mesh_pkg}/base_motor_holder_so101_v1.stl"/></geometry>
+    </collision>
+    <visual>
+      <origin xyz="-0.00636471 -8.97657e-09 -0.0024" rpy="1.5708 0 1.5708"/>
+      <geometry><mesh filename="${mesh_pkg}/base_so101_v2.stl"/></geometry>
+      <material name="3d_printed"/>
+    </visual>
+    <collision>
+      <origin xyz="-0.00636471 -8.97657e-09 -0.0024" rpy="1.5708 0 1.5708"/>
+      <geometry><mesh filename="${mesh_pkg}/base_so101_v2.stl"/></geometry>
+    </collision>
+    <visual>
+      <origin xyz="0.0263353 -8.97657e-09 0.0437" rpy="0 0 0"/>
+      <geometry><mesh filename="${mesh_pkg}/sts3215_03a_v1.stl"/></geometry>
+      <material name="sts3215"/>
+    </visual>
+    <collision>
+      <origin xyz="0.0263353 -8.97657e-09 0.0437" rpy="0 0 0"/>
+      <geometry><mesh filename="${mesh_pkg}/sts3215_03a_v1.stl"/></geometry>
+    </collision>
+    <visual>
+      <origin xyz="-0.0309827 -0.000199441 0.0474" rpy="1.5708 0 1.5708"/>
+      <geometry><mesh filename="${mesh_pkg}/waveshare_mounting_plate_so101_v2.stl"/></geometry>
+      <material name="3d_printed"/>
+    </visual>
+    <collision>
+      <origin xyz="-0.0309827 -0.000199441 0.0474" rpy="1.5708 0 1.5708"/>
+      <geometry><mesh filename="${mesh_pkg}/waveshare_mounting_plate_so101_v2.stl"/></geometry>
+    </collision>
+  </link>
+  <!-- ── Joint 1: shoulder_pan ─────────────────────────────── -->
+  <joint name="shoulder_pan" type="revolute">
     <parent link="base_link"/>
-    <child  link="link1"/>
-    <origin xyz="0 0 0.05" rpy="0 0 0"/>
-    <axis xyz="0 0 1"/>
-    <limit lower="${-pi}" upper="${pi}" effort="10" velocity="2.0"/>
-    <dynamics damping="0.1" friction="0.05"/>
-  </joint>
-  <link name="link1">
-    <visual>
-      <origin xyz="0 0 0.04" rpy="0 0 0"/>
-      <geometry><box size="0.05 0.05 0.08"/></geometry>
-      <material name="light_grey"/>
-    </visual>
-    <collision>
-      <origin xyz="0 0 0.04" rpy="0 0 0"/>
-      <geometry><box size="0.05 0.05 0.08"/></geometry>
-    </collision>
-    <xacro:box_inertia m="0.2" x="0.05" y="0.05" z="0.08"/>
-  </link>
-  <!-- ───────── Joint 2: Shoulder pitch ───────── -->
-  <joint name="joint2" type="revolute">
-    <parent link="link1"/>
-    <child  link="link2"/>
-    <origin xyz="0 0 0.085" rpy="0 0 0"/>
-    <axis xyz="0 1 0"/>
-    <limit lower="${-pi/2}" upper="${pi/2}" effort="10" velocity="2.0"/>
-    <dynamics damping="0.1" friction="0.05"/>
-  </joint>
-  <link name="link2">
-    <visual>
-      <origin xyz="0 0 0.065" rpy="0 0 0"/>
-      <geometry><box size="0.04 0.04 0.13"/></geometry>
-      <material name="white"/>
-    </visual>
-    <collision>
-      <origin xyz="0 0 0.065" rpy="0 0 0"/>
-      <geometry><box size="0.04 0.04 0.13"/></geometry>
-    </collision>
-    <xacro:box_inertia m="0.18" x="0.04" y="0.04" z="0.13"/>
-  </link>
-  <!-- ───────── Joint 3: Elbow pitch ───────── -->
-  <joint name="joint3" type="revolute">
-    <parent link="link2"/>
-    <child  link="link3"/>
-    <origin xyz="0 0 0.13" rpy="0 0 0"/>
-    <axis xyz="0 1 0"/>
-    <limit lower="${-pi*2/3}" upper="${pi*2/3}" effort="8" velocity="2.0"/>
-    <dynamics damping="0.1" friction="0.05"/>
-  </joint>
-  <link name="link3">
-    <visual>
-      <origin xyz="0 0 0.055" rpy="0 0 0"/>
-      <geometry><box size="0.038 0.038 0.11"/></geometry>
-      <material name="light_grey"/>
-    </visual>
-    <collision>
-      <origin xyz="0 0 0.055" rpy="0 0 0"/>
-      <geometry><box size="0.038 0.038 0.11"/></geometry>
-    </collision>
-    <xacro:box_inertia m="0.14" x="0.038" y="0.038" z="0.11"/>
-  </link>
-  <!-- ───────── Joint 4: Wrist pitch ───────── -->
-  <joint name="joint4" type="revolute">
-    <parent link="link3"/>
-    <child  link="link4"/>
-    <origin xyz="0 0 0.11" rpy="0 0 0"/>
-    <axis xyz="0 1 0"/>
-    <limit lower="${-pi/2}" upper="${pi/2}" effort="5" velocity="3.0"/>
-    <dynamics damping="0.05" friction="0.02"/>
-  </joint>
-  <link name="link4">
-    <visual>
-      <origin xyz="0 0 0.035" rpy="0 0 0"/>
-      <geometry><box size="0.035 0.035 0.07"/></geometry>
-      <material name="white"/>
-    </visual>
-    <collision>
-      <origin xyz="0 0 0.035" rpy="0 0 0"/>
-      <geometry><box size="0.035 0.035 0.07"/></geometry>
-    </collision>
-    <xacro:box_inertia m="0.10" x="0.035" y="0.035" z="0.07"/>
-  </link>
-  <!-- ───────── Joint 5: Wrist roll ───────── -->
-  <joint name="joint5" type="revolute">
-    <parent link="link4"/>
-    <child  link="link5"/>
-    <origin xyz="0 0 0.07" rpy="0 0 0"/>
-    <axis xyz="0 0 1"/>
-    <limit lower="${-pi}" upper="${pi}" effort="5" velocity="3.0"/>
-    <dynamics damping="0.05" friction="0.02"/>
-  </joint>
-  <link name="link5">
-    <visual>
-      <origin xyz="0 0 0.025" rpy="0 0 0"/>
-      <geometry><cylinder radius="0.020" length="0.05"/></geometry>
-      <material name="dark_grey"/>
-    </visual>
-    <collision>
-      <origin xyz="0 0 0.025" rpy="0 0 0"/>
-      <geometry><cylinder radius="0.020" length="0.05"/></geometry>
-    </collision>
-    <xacro:box_inertia m="0.06" x="0.04" y="0.04" z="0.05"/>
-  </link>
-  <!-- ───────── Gripper base ───────── -->
-  <joint name="gripper_base_joint" type="fixed">
-    <parent link="link5"/>
-    <child  link="gripper_base"/>
-    <origin xyz="0 0 0.05" rpy="0 0 0"/>
-  </joint>
-  <link name="gripper_base">
-    <visual>
-      <origin xyz="0 0 0.01" rpy="0 0 0"/>
-      <geometry><box size="0.06 0.025 0.02"/></geometry>
-      <material name="dark_grey"/>
-    </visual>
-    <collision>
-      <origin xyz="0 0 0.01" rpy="0 0 0"/>
-      <geometry><box size="0.06 0.025 0.02"/></geometry>
-    </collision>
-    <xacro:box_inertia m="0.05" x="0.06" y="0.025" z="0.02"/>
-  </link>
-  <!-- ───────── Gripper finger left ───────── -->
-  <joint name="gripper_left_joint" type="prismatic">
-    <parent link="gripper_base"/>
-    <child  link="gripper_left"/>
-    <origin xyz="-0.015 0 0.02" rpy="0 0 0"/>
-    <axis xyz="1 0 0"/>
-    <limit lower="-0.025" upper="0.0" effort="5" velocity="0.1"/>
-    <dynamics damping="0.05" friction="0.01"/>
-  </joint>
-  <link name="gripper_left">
-    <visual>
-      <origin xyz="0 0 0.02" rpy="0 0 0"/>
-      <geometry><box size="0.01 0.018 0.04"/></geometry>
-      <material name="orange"/>
-    </visual>
-    <collision>
-      <origin xyz="0 0 0.02" rpy="0 0 0"/>
-      <geometry><box size="0.01 0.018 0.04"/></geometry>
-    </collision>
-    <xacro:box_inertia m="0.02" x="0.01" y="0.018" z="0.04"/>
-  </link>
-  <!-- ───────── Gripper finger right (mimic) ───────── -->
-  <joint name="gripper_right_joint" type="prismatic">
-    <parent link="gripper_base"/>
-    <child  link="gripper_right"/>
-    <origin xyz="0.015 0 0.02" rpy="0 0 0"/>
-    <axis xyz="-1 0 0"/>
-    <limit lower="-0.025" upper="0.0" effort="5" velocity="0.1"/>
-    <mimic joint="gripper_left_joint" multiplier="1.0" offset="0.0"/>
-    <dynamics damping="0.05" friction="0.01"/>
-  </joint>
-  <link name="gripper_right">
-    <visual>
-      <origin xyz="0 0 0.02" rpy="0 0 0"/>
-      <geometry><box size="0.01 0.018 0.04"/></geometry>
-      <material name="orange"/>
-    </visual>
-    <collision>
-      <origin xyz="0 0 0.02" rpy="0 0 0"/>
-      <geometry><box size="0.01 0.018 0.04"/></geometry>
-    </collision>
-    <xacro:box_inertia m="0.02" x="0.01" y="0.018" z="0.04"/>
-  </link>
-  <!-- ───────── Tool-center point ───────── -->
+    <child  link="shoulder_link"/>
+    <origin xyz="0.0388353 -8.97657e-09 0.0624" rpy="3.14159 0 -3.14159"/>
+    <axis xyz="0 0 1"/>
+    <limit lower="-1.91986" upper="1.91986" effort="10" velocity="2.0"/>
+    <dynamics damping="0.6" friction="0.052"/>
+  </joint>
+  <!-- ── shoulder_link ─────────────────────────────────────── -->
+  <link name="shoulder_link">
+    <inertial>
+      <origin xyz="-0.0307604 -1.66727e-05 -0.0252713" rpy="0 0 0"/>
+      <mass value="0.100006"/>
+      <inertia ixx="8.3759e-05" ixy="7.55525e-08" ixz="-1.16342e-06"
+               iyy="8.10403e-05" iyz="1.54663e-07" izz="2.39783e-05"/>
+    </inertial>
+    <visual>
+      <origin xyz="-0.0303992 0.000422241 -0.0417" rpy="1.5708 1.5708 0"/>
+      <geometry><mesh filename="${mesh_pkg}/sts3215_03a_v1.stl"/></geometry>
+      <material name="sts3215"/>
+    </visual>
+    <collision>
+      <origin xyz="-0.0303992 0.000422241 -0.0417" rpy="1.5708 1.5708 0"/>
+      <geometry><mesh filename="${mesh_pkg}/sts3215_03a_v1.stl"/></geometry>
+    </collision>
+    <visual>
+      <origin xyz="-0.0675992 -0.000177759 0.0158499" rpy="1.5708 -1.5708 0"/>
+      <geometry><mesh filename="${mesh_pkg}/motor_holder_so101_base_v1.stl"/></geometry>
+      <material name="3d_printed"/>
+    </visual>
+    <collision>
+      <origin xyz="-0.0675992 -0.000177759 0.0158499" rpy="1.5708 -1.5708 0"/>
+      <geometry><mesh filename="${mesh_pkg}/motor_holder_so101_base_v1.stl"/></geometry>
+    </collision>
+    <visual>
+      <origin xyz="0.0122008 2.22413e-05 0.0464" rpy="-1.5708 0 0"/>
+      <geometry><mesh filename="${mesh_pkg}/rotation_pitch_so101_v1.stl"/></geometry>
+      <material name="3d_printed"/>
+    </visual>
+    <collision>
+      <origin xyz="0.0122008 2.22413e-05 0.0464" rpy="-1.5708 0 0"/>
+      <geometry><mesh filename="${mesh_pkg}/rotation_pitch_so101_v1.stl"/></geometry>
+    </collision>
+  </link>
+  <!-- ── Joint 2: shoulder_lift ────────────────────────────── -->
+  <joint name="shoulder_lift" type="revolute">
+    <parent link="shoulder_link"/>
+    <child  link="upper_arm_link"/>
+    <origin xyz="-0.0303992 -0.0182778 -0.0542" rpy="-1.5708 -1.5708 0"/>
+    <axis xyz="0 0 1"/>
+    <limit lower="-1.74533" upper="1.74533" effort="10" velocity="2.0"/>
+    <dynamics damping="0.6" friction="0.052"/>
+  </joint>
+  <!-- ── upper_arm_link ────────────────────────────────────── -->
+  <link name="upper_arm_link">
+    <inertial>
+      <origin xyz="-0.0898471 -0.00838224 0.0184089" rpy="0 0 0"/>
+      <mass value="0.103"/>
+      <inertia ixx="4.08002e-05" ixy="-1.97819e-05" ixz="-4.03016e-08"
+               iyy="0.000147318" iyz="8.97326e-09" izz="0.000142487"/>
+    </inertial>
+    <visual>
+      <origin xyz="-0.11257 -0.0155 0.0187" rpy="-3.14159 0 -1.5708"/>
+      <geometry><mesh filename="${mesh_pkg}/sts3215_03a_v1.stl"/></geometry>
+      <material name="sts3215"/>
+    </visual>
+    <collision>
+      <origin xyz="-0.11257 -0.0155 0.0187" rpy="-3.14159 0 -1.5708"/>
+      <geometry><mesh filename="${mesh_pkg}/sts3215_03a_v1.stl"/></geometry>
+    </collision>
+    <visual>
+      <origin xyz="-0.065085 0.012 0.0182" rpy="3.14159 0 0"/>
+      <geometry><mesh filename="${mesh_pkg}/upper_arm_so101_v1.stl"/></geometry>
+      <material name="3d_printed"/>
+    </visual>
+    <collision>
+      <origin xyz="-0.065085 0.012 0.0182" rpy="3.14159 0 0"/>
+      <geometry><mesh filename="${mesh_pkg}/upper_arm_so101_v1.stl"/></geometry>
+    </collision>
+  </link>
+  <!-- ── Joint 3: elbow_flex ───────────────────────────────── -->
+  <joint name="elbow_flex" type="revolute">
+    <parent link="upper_arm_link"/>
+    <child  link="lower_arm_link"/>
+    <origin xyz="-0.11257 -0.028 0" rpy="0 0 1.5708"/>
+    <axis xyz="0 0 1"/>
+    <limit lower="-1.69" upper="1.69" effort="10" velocity="2.0"/>
+    <dynamics damping="0.6" friction="0.052"/>
+  </joint>
+  <!-- ── lower_arm_link ────────────────────────────────────── -->
+  <link name="lower_arm_link">
+    <inertial>
+      <origin xyz="-0.0980701 0.00324376 0.0182831" rpy="0 0 0"/>
+      <mass value="0.104"/>
+      <inertia ixx="2.87438e-05" ixy="7.41152e-06" ixz="1.26409e-06"
+               iyy="0.000159844" iyz="-4.90188e-08" izz="0.00014529"/>
+    </inertial>
+    <visual>
+      <origin xyz="-0.0648499 -0.032 0.0182" rpy="3.14159 0 0"/>
+      <geometry><mesh filename="${mesh_pkg}/under_arm_so101_v1.stl"/></geometry>
+      <material name="3d_printed"/>
+    </visual>
+    <collision>
+      <origin xyz="-0.0648499 -0.032 0.0182" rpy="3.14159 0 0"/>
+      <geometry><mesh filename="${mesh_pkg}/under_arm_so101_v1.stl"/></geometry>
+    </collision>
+    <visual>
+      <origin xyz="-0.0648499 -0.032 0.018" rpy="-3.14159 0 0"/>
+      <geometry><mesh filename="${mesh_pkg}/motor_holder_so101_wrist_v1.stl"/></geometry>
+      <material name="3d_printed"/>
+    </visual>
+    <collision>
+      <origin xyz="-0.0648499 -0.032 0.018" rpy="-3.14159 0 0"/>
+      <geometry><mesh filename="${mesh_pkg}/motor_holder_so101_wrist_v1.stl"/></geometry>
+    </collision>
+    <visual>
+      <origin xyz="-0.1224 0.0052 0.0187" rpy="-3.14159 0 -3.14159"/>
+      <geometry><mesh filename="${mesh_pkg}/sts3215_03a_v1.stl"/></geometry>
+      <material name="sts3215"/>
+    </visual>
+    <collision>
+      <origin xyz="-0.1224 0.0052 0.0187" rpy="-3.14159 0 -3.14159"/>
+      <geometry><mesh filename="${mesh_pkg}/sts3215_03a_v1.stl"/></geometry>
+    </collision>
+  </link>
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